File: FPGA_Power.sch (KiCad schematic (older format))
At the start: 1 part, among them U1 XA7Z020-1CLG400Q

Commit message: Completed FPGA power sheet completed USB3 completed FPGA config
Parts:
- added C?: C_Small, Capacitor_SMD:C_0603_1608Metric_Pad1.08x0.95mm_HandSolder, symbol Device:C_Small
- added C?: C_Polarized_Small, Capacitor_Tantalum_SMD:CP_EIA-1608-10_AVX-L_Pad1.25x1.05mm_HandSolder, symbol Device:C_Polarized_Small
- added C?: C_Small, symbol Device:C_Small
- added C? (x38): 470nF, Capacitor_SMD:C_0603_1608Metric_Pad1.08x0.95mm_HandSolder, symbol Device:C_Small
- added C? (x23): 4.7uF, Capacitor_SMD:C_0603_1608Metric_Pad1.08x0.95mm_HandSolder, symbol Device:C_Small
- added C? (x9): 100uF, Capacitor_SMD:C_1210_3225Metric_Pad1.33x2.70mm_HandSolder, symbol Device:C_Small
- added C?: 47uF, Capacitor_SMD:C_1210_3225Metric_Pad1.33x2.70mm_HandSolder, symbol Device:C_Small
- added C?: 10uF, Capacitor_SMD:C_0805_2012Metric_Pad1.18x1.45mm_HandSolder, symbol Device:C_Small
- added FB?: MPZ2012S601AT000, digikey-footprints:0805, symbol dk_Ferrite-Beads-and-Chips:MPZ2012S601AT000
- added R?: R_Small_US, Resistor_SMD:R_0603_1608Metric_Pad0.98x0.95mm_HandSolder, symbol Device:R_Small_US
- added R?: 0, Resistor_SMD:R_0603_1608Metric_Pad0.98x0.95mm_HandSolder, symbol Device:R_Small_US
Connections:
- net labels added: GNDD, VCC1V0, VCC1V35, VCC1V8, VCC3V3, VCCPLL
- wire segments 0 -> 270
Other:
- moved on the sheet: U1H, U1I
