File: Digital_Board.kicad_pcb (KiCad board)
At the start: 2 copper layers, 744 parts, among them IC1 M24M02-DRMN6TP, IC10 AD9726BSVZ, IC11 LTC2387CUH-18#PBF, IC12 LTC2387CUH-18#PBF, IC13 LTC2387CUH-18#PBF, IC14 SP3232EEN-L_TR, IC15 LTM8078IY#PBF, IC17 SN74LVC3G14DCUR, IC2 ADR127BUJZ-REEL7, IC3 TXS02612RTWR, IC4 USB3320C-EZK, IC5 LM5116MHX_NOPB, IC6 LM5116MHX_NOPB, IC7 M24M02-DRMN6TP, IC9 CY7C1062GE30-10BGXI, J1 104031-0811, J10 Screw_Terminal_01x02, J12 USB3_B, J21 5747840-6, J3 Conn_01x02, J5 BoardEdge_of_HSEC8-140-01-L-P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, J6 BoardEdge_of_HSEC8-140-01-L-P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, J7 UE27AC54100, J8 0475890001, J9 Screw_Terminal_01x03, Q1 FDS9926A, Q2 MCH3481-TL-W, Q3 FDV301N, Q4 CSD18534Q5A, Q5 CSD18540Q5B, Q6 CSD18534Q5A, Q7 CSD18540Q5B, Q8 FDV301N, U1 XA7Z020-1CLG400Q, U11 WE-TVS-82400102, U12 NCP1117ST33T3G, U13 MIC23150, U16 TCA9406DC, U17 TXS0108EPW, U18 TXS0108EPW, U2 AS4C256M16D3LC-12BCN, U3 AS4C256M16D3LC-12BCN, U4 Si5344A-D, U5 ADP5052ACPZ-R7, U6 TPS2051BDBVR, U7 DP83869HMRGZT, U8 DS3231S#, U9 BU2032SM-HD-G, Y1 XRCGE25M000FBA1AR0, Y2 CX3225SB48000D0FPJC1, Y3 19.2Mhz

Commit message: Corrected PCB import errors
Parts:
- added C111: 150uF, Capacitor_Tantalum_SMD:CP_EIA-7343-30_AVX-N, F.Cu at (547.4, 203.2)
- added D11: LED_Small, LED_SMD:LED_0603_1608Metric, F.Cu at (526.2, 183.4)
- added D3: LED_Small, LED_SMD:LED_0603_1608Metric, F.Cu at (478.7, 196.6)
- added IC8: TPD4E05U06QDQARQ1, GM_SON:DQA_R-PUSON-N10_, F.Cu at (521.4, 189.6)
- added J15: Conn_01x04, Connector_PinHeader_2.54mm:PinHeader_1x04_P2.54mm_Vertical, F.Cu at (540.5, 169.6)
- added J16: Conn_01x04, Connector_PinHeader_2.54mm:PinHeader_1x04_P2.54mm_Vertical, F.Cu at (535.8, 169.6)
- added J17: Conn_01x06, Connector_PinHeader_2.54mm:PinHeader_1x06_P2.54mm_Vertical, F.Cu at (521.9, 169.6)
- added J18: Conn_01x04, Connector_PinHeader_2.54mm:PinHeader_1x04_P2.54mm_Vertical, F.Cu at (531.2, 169.6)
- added J19: Conn_01x05, Connector_PinHeader_2.54mm:PinHeader_1x05_P2.54mm_Vertical, F.Cu at (526.5, 169.6)
- added J2: Conn_01x06, Connector_PinHeader_2.54mm:PinHeader_1x06_P2.54mm_Vertical, F.Cu at (474.3, 197.7)
- added J20: RJMG2012211A0FR, GM_Connectors:RJMG2012211A0FR, F.Cu at (493.4, 183.9)
- added L1: 3.3uH, Inductor_SMD:L_Coilcraft_XAL60xx_6.36x6.56mm, F.Cu at (527.9, 199.4)
- added L2: 1uH, Inductor_SMD:L_Coilcraft_XAL60xx_6.36x6.56mm, F.Cu at (520.0, 199.4)
- added L3: 6.8uH, Inductor_SMD:L_Coilcraft_XAL60xx_6.36x6.56mm, F.Cu at (512.1, 207.5)
- added L4: 6.8uH, Inductor_SMD:L_Coilcraft_XAL60xx_6.36x6.56mm, F.Cu at (512.1, 199.4)
- added L7: 1uH, Inductor_SMD:L_Coilcraft_XAL60xx_6.36x6.56mm, F.Cu at (546.4, 192.5)
- added TP1: TestPoint, TestPoint:TestPoint_Pad_2.0x2.0mm, F.Cu at (556.9, 169.3)
- renumbered C29 to C1, C38 to C10, C142 to C100, C143 to C101, C144 to C102, C145 to C103, C146 to C104, C147 to C105, C148 to C106, C149 to C107, C150 to C108, C151 to C109, C39 to C11, C152 to C110, C154 to C112, C155 to C113, C2 to C114, C3 to C115, C45 to C116, C46 to C117, C47 to C118, C48 to C119, C40 to C12, C4 to C120, C49 to C121, C5 to C122, C6 to C123, C50 to C124, C7 to C125, C8 to C126, C9 to C127, C10 to C128, C11 to C129, C41 to C13, C12 to C130, C13 to C131, C14 to C132, C51 to C133, C15 to C134, C16 to C135, C17 to C136, C18 to C137, C19 to C138, C20 to C139, C52 to C14, C21 to C140, C22 to C141, C23 to C142, C24 to C143, C25 to C144, C26 to C145, C162 to C146, C163 to C147, C164 to C148, C165 to C149, C53 to C15, C166 to C150, C167 to C151, C168 to C152, C169 to C153, C170 to C154, C171 to C155, C172 to C156, C173 to C157, C174 to C158, C175 to C159, C55 to C16, C176 to C160, C177 to C161, C178 to C162, C179 to C163, C180 to C164, C181 to C165, C182 to C166, C183 to C167, C184 to C168, C185 to C169, C56 to C17, C54 to C170, C186 to C171, C190 to C172, C191 to C173, C192 to C174, C193 to C175, C194 to C176, C195 to C177, C196 to C178, C200 to C179, C57 to C18, C201 to C180, C202 to C181, C203 to C182, C204 to C183, C205 to C184, C206 to C185, C207 to C186, C208 to C187, C209 to C188, C210 to C189, C58 to C19, C211 to C190, C212 to C191, C213 to C192, C214 to C193, C215 to C194, C216 to C195, C217 to C196, C218 to C197, C219 to C198, C220 to C199, C30 to C2, C59 to C20, C221 to C200, C222 to C201, C223 to C202, C224 to C203, C225 to C204, C226 to C205, C227 to C206, C228 to C207, C229 to C208, C230 to C209, C60 to C21, C231 to C210, C232 to C211, C233 to C212, C234 to C213, C235 to C214, C236 to C215, C237 to C216, C238 to C217, C239 to C218, C240 to C219, C61 to C22, C241 to C220, C242 to C221, C243 to C222, C244 to C223, C245 to C224, C246 to C225, C247 to C226, C248 to C227, C249 to C228, C250 to C229, C62 to C23, C251 to C230, C252 to C231, C253 to C232, C254 to C233, C255 to C234, C256 to C235, C257 to C236, C260 to C237, C261 to C238, C262 to C239, C63 to C24, C263 to C240, C267 to C241, C268 to C242, C269 to C243, C270 to C244, C271 to C245, C272 to C246, C276 to C247, C277 to C248, C278 to C249, C64 to C25, C279 to C250, C280 to C251, C281 to C252, C282 to C253, C283 to C254, C284 to C255, C285 to C256, C286 to C257, C287 to C258, C288 to C259, C65 to C26, C289 to C260, C290 to C261, C291 to C262, C292 to C263, C293 to C264, C294 to C265, C298 to C266, C299 to C267, C300 to C268, C301 to C269, C66 to C27, C302 to C270, C303 to C271, C304 to C272, C305 to C273, C309 to C274, C310 to C275, C311 to C276, C312 to C277, C313 to C278, C314 to C279, C67 to C28, C315 to C280, C316 to C281, C320 to C282, C321 to C283, C322 to C284, C323 to C285, C324 to C286, C325 to C287, C326 to C288, C327 to C289, C68 to C29, C334 to C290, C335 to C291, C336 to C292, C337 to C293, C338 to C294, C339 to C295, C340 to C296, C341 to C297, C342 to C298, C343 to C299, C31 to C3, C69 to C30, C344 to C300, C345 to C301, C346 to C302, C347 to C303, C348 to C304, C349 to C305, C350 to C306, C351 to C307, C352 to C308, C353 to C309, C70 to C31, C354 to C310, C355 to C311, C356 to C312, C357 to C313, C358 to C314, C359 to C315, C360 to C316, C361 to C317, C362 to C318, C363 to C319, C71 to C32, C364 to C320, C365 to C321, C366 to C322, C367 to C323, C368 to C324, C369 to C325, C370 to C326, C371 to C327, C372 to C328, C373 to C329, C72 to C33, C374 to C330, C375 to C331, C376 to C332, C377 to C333, C378 to C334, C379 to C335, C380 to C336, C381 to C337, C382 to C338, C383 to C339, C73 to C34, C384 to C340, C385 to C341, C386 to C342, C387 to C343, C388 to C344, C389 to C345, C390 to C346, C391 to C347, C392 to C348, C393 to C349, C74 to C35, C394 to C350, C395 to C351, C396 to C352, C397 to C353, C398 to C354, C399 to C355, C400 to C356, C401 to C357, C402 to C358, C403 to C359, C75 to C36, C404 to C360, C405 to C361, C406 to C362, C407 to C363, C408 to C364, C409 to C365, C410 to C366, C411 to C367, C412 to C368, C413 to C369, C76 to C37, C414 to C370, C415 to C371, C416 to C372, C417 to C373, C418 to C374, C419 to C375, C420 to C376, C421 to C377, C422 to C378, C423 to C379, C77 to C38, C424 to C380, C42 to C381, C43 to C382, C44 to C383, C425 to C384, C426 to C385, C427 to C386, C428 to C387, C429 to C388, C431 to C389, C78 to C39, C329 to C390, C330 to C391, C331 to C392, C332 to C393, C333 to C394, C32 to C4, C79 to C40, C80 to C41, C81 to C42, C82 to C43, C83 to C44, C84 to C45, C85 to C46, C86 to C47, C87 to C48, C88 to C49, C33 to C5, C89 to C50, C90 to C51, C91 to C52, C92 to C53, C93 to C54, C94 to C55, C95 to C56, C96 to C57, C97 to C58, C98 to C59, C34 to C6, C99 to C60, C100 to C61, C101 to C62, C102 to C63, C103 to C64, C104 to C65, C105 to C66, C106 to C67, C107 to C68, C108 to C69, C35 to C7, C109 to C70, C110 to C71, C111 to C72, C112 to C73, C113 to C74, C114 to C75, C115 to C76, C116 to C77, C117 to C78, C118 to C79, C36 to C8, C122 to C80, C123 to C81, C124 to C82, C125 to C83, C126 to C84, C127 to C85, C128 to C86, C129 to C87, C130 to C88, C131 to C89, C37 to C9, C132 to C90, C133 to C91, C134 to C92, C135 to C93, C136 to C94, C137 to C95, C138 to C96, C139 to C97, C140 to C98, C141 to C99, D6 to D1, D11 to D10, D13 to D12, D7 to D2, D1 to D4, D2 to D5, D3 to D6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
Connections:
- net /RTC_FAN/RTC_SCL renamed /I2C2_SCL
- C100 pad 1: (no net) -> /FDAC_CLKIN_N
- C101 pad 1: (no net) -> /Clock_Gen/CLK_OUT1_N
- C102 pad 1: (no net) -> /Clock_Gen/CLK_OUT2_N
- C103 pad 1: (no net) -> /Clock_Gen/CLK_OUT3_N
- C137 pad 2: (no net) -> Net-(C137-Pad2)
- C138 pad 1: (no net) -> Net-(C138-Pad1)
- C177 pad 1: (no net) -> Net-(C177-Pad1)
- C178 pad 1: (no net) -> Net-(C178-Pad1)
- C385 pad 1: (no net) -> Net-(C385-Pad1)
- C386 pad 1: (no net) -> Net-(C386-Pad1)
- C387 pad 1: (no net) -> Net-(C387-Pad1)
- C388 pad 1: (no net) -> Net-(C388-Pad1)
- C83 pad 2: (no net) -> /Clock_Gen/CLK_IN0_P
- C84 pad 2: (no net) -> /Clock_Gen/CLK_IN0_N
- C85 pad 2: (no net) -> /Clock_Gen/CLK_IN1_P
- C86 pad 2: (no net) -> /Clock_Gen/CLK_IN1_N
- C87 pad 2: (no net) -> /Clock_Gen/CLK_IN2_P
- C88 pad 2: (no net) -> /Clock_Gen/CLK_IN2_N
- C89 pad 2: (no net) -> /Clock_Gen/CLK_IN3_P
- C90 pad 2: (no net) -> /Clock_Gen/CLK_IN3_N
- C95 pad 1: (no net) -> /FDAC_CLKIN_P
- C96 pad 1: (no net) -> /Clock_Gen/CLK_OUT1_P
- C97 pad 1: (no net) -> /Clock_Gen/CLK_OUT2_P
- C98 pad 1: (no net) -> /Clock_Gen/CLK_OUT3_P
- D4 pad 1: /RTC_FAN/12VIN -> /12V
- D5 pad 2: (no net) -> Net-(D5-Pad2)
- IC1 pad 1: (no net) -> /FPGA_Config/SD_DAT2
- IC1 pad 10: (no net) -> Net-(IC1-Pad10)
- IC1 pad 12: (no net) -> Net-(IC1-Pad12)
- IC1 pad 13: (no net) -> Net-(IC1-Pad13)
- IC1 pad 14: (no net) -> Net-(IC1-Pad14)
- IC1 pad 15: (no net) -> Net-(IC1-Pad15)
- IC1 pad 3: (no net) -> /FPGA_Config/SD_DAT3
- IC1 pad 4: (no net) -> /FPGA_Config/SD_CMD
- IC1 pad 6: (no net) -> /FPGA_Config/SD_DAT0
- IC1 pad 7: (no net) -> /FPGA_Config/SD_DAT1
- IC1 pad 8: (no net) -> Net-(IC1-Pad8)
- IC1 pad 9: (no net) -> /FPGA_Config/SD_CLK
- IC10 pad 10: (no net) -> /AWG/FDAC_DB15_P
- IC10 pad 11: (no net) -> /AWG/FDAC_DB15_N
- IC10 pad 12: (no net) -> /AWG/FDAC_DB14_P
- IC10 pad 13: (no net) -> /AWG/FDAC_DB14_N
- IC10 pad 14: (no net) -> /AWG/FDAC_DB13_P
- IC10 pad 15: (no net) -> /AWG/FDAC_DB13_N
- IC10 pad 16: (no net) -> /AWG/FDAC_DB12_P
- IC10 pad 17: (no net) -> /AWG/FDAC_DB12_N
- IC10 pad 18: (no net) -> /AWG/FDAC_DB11_P
- IC10 pad 19: (no net) -> /AWG/FDAC_DB11_N
- IC10 pad 22: (no net) -> /AWG/FDAC_DB10_P
- IC10 pad 23: (no net) -> /AWG/FDAC_DB10_N
- IC10 pad 24: (no net) -> /AWG/FDAC_DB9_P
- IC10 pad 25: (no net) -> /AWG/FDAC_DB9_N
- IC10 pad 26: (no net) -> /AWG/FDAC_DB8_P
- IC10 pad 27: (no net) -> /AWG/FDAC_DB8_N
- IC10 pad 28: (no net) -> /AWG/FDAC_DCLK_OUT_P
- IC10 pad 29: (no net) -> /AWG/FDAC_DCLK_OUT_N
- IC10 pad 32: (no net) -> /AWG/FDAC_DCLK_IN_P
- IC10 pad 33: (no net) -> /AWG/FDAC_DCLK_IN_N
- IC10 pad 34: (no net) -> /AWG/FDAC_DB7_P
- IC10 pad 35: (no net) -> /AWG/FDAC_DB7_N
- IC10 pad 36: (no net) -> /AWG/FDAC_DB6_P
- IC10 pad 37: (no net) -> /AWG/FDAC_DB6_N
- IC10 pad 38: (no net) -> /AWG/FDAC_DB5_P
- IC10 pad 39: (no net) -> /AWG/FDAC_DB5_N
- IC10 pad 42: (no net) -> /AWG/FDAC_DB4_P
- IC10 pad 43: (no net) -> /AWG/FDAC_DB4_N
- IC10 pad 44: (no net) -> /AWG/FDAC_DB3_P
- IC10 pad 45: (no net) -> /AWG/FDAC_DB3_N
- IC10 pad 46: (no net) -> /AWG/FDAC_DB2_P
- IC10 pad 47: (no net) -> /AWG/FDAC_DB2_N
- IC10 pad 48: (no net) -> /AWG/FDAC_DB1_P
- IC10 pad 49: (no net) -> /AWG/FDAC_DB1_N
- IC10 pad 5: (no net) -> /AWG/FDAC_CLKIN_P
- IC10 pad 50: (no net) -> /AWG/FDAC_DB0_P
- IC10 pad 51: (no net) -> /AWG/FDAC_DB0_N
- IC10 pad 54: (no net) -> /AWG/FDAC_SDO
- IC10 pad 55: (no net) -> /AWG/FDAC_SDI
- IC10 pad 56: (no net) -> /AWG/FDAC_CLK
- IC10 pad 57: (no net) -> /AWG/FDAC_CS
- IC10 pad 58: (no net) -> Net-(IC10-Pad58)
- IC10 pad 6: (no net) -> /AWG/FDAC_CLKIN_N
- IC10 pad 70: (no net) -> Net-(IC10-Pad70)
- IC10 pad 71: (no net) -> Net-(IC10-Pad71)
- IC11 pad 15: (no net) -> Net-(IC11-Pad15)
- IC11 pad 16: (no net) -> Net-(IC11-Pad16)
- IC11 pad 17: (no net) -> /ADC/ADC1_DA_N
- IC11 pad 18: (no net) -> /ADC/ADC1_DA_P
- IC11 pad 19: (no net) -> /ADC/ADC1_DCO_N
- IC11 pad 2: (no net) -> Net-(IC11-Pad2)
- IC11 pad 20: (no net) -> /ADC/ADC1_DCO_P
- IC11 pad 23: (no net) -> /ADC/ADC1_CLK_N
- IC11 pad 24: (no net) -> /ADC/ADC1_CLK_P
- IC11 pad 3: (no net) -> Net-(IC11-Pad3)
- IC12 pad 15: (no net) -> Net-(IC12-Pad15)
- IC12 pad 16: (no net) -> Net-(IC12-Pad16)
- IC12 pad 17: (no net) -> /ADC/ADC2_DA_N
- IC12 pad 18: (no net) -> /ADC/ADC2_DA_P
- IC12 pad 19: (no net) -> /ADC/ADC2_DCO_N
- IC12 pad 2: (no net) -> Net-(IC12-Pad2)
- IC12 pad 20: (no net) -> /ADC/ADC2_DCO_P
- IC12 pad 23: (no net) -> /ADC/ADC2_CLK_N
- IC12 pad 24: (no net) -> /ADC/ADC2_CLK_P
- IC12 pad 3: (no net) -> Net-(IC12-Pad3)
- IC13 pad 15: (no net) -> Net-(IC13-Pad15)
- IC13 pad 16: (no net) -> Net-(IC13-Pad16)
- IC13 pad 17: (no net) -> /ADC/ADC3_DA_N
- IC13 pad 18: (no net) -> /ADC/ADC3_DA_P
- IC13 pad 19: (no net) -> /ADC/ADC3_DCO_N
- IC13 pad 2: (no net) -> Net-(IC13-Pad2)
- IC13 pad 20: (no net) -> /ADC/ADC3_DCO_P
- IC13 pad 23: (no net) -> /ADC/ADC3_CLK_N
- IC13 pad 24: (no net) -> /ADC/ADC3_CLK_P
- IC13 pad 3: (no net) -> Net-(IC13-Pad3)
- IC14 pad D1: (no net) -> Net-(IC14-PadD1)
- IC18 pad 10: (no net) -> /RS232_Port/RS232_RTS
- IC18 pad 11: (no net) -> /FPGA_Banks/RS232_TX
- IC18 pad 12: (no net) -> /FPGA_Banks/RS232_RX
- IC18 pad 9: (no net) -> /RS232_Port/RS232_CTS
- IC2 pad 12: (no net) -> Net-(IC2-Pad12)
- IC2 pad 15: (no net) -> Net-(IC2-Pad15)
- IC2 pad 16: (no net) -> Net-(IC2-Pad16)
- IC2 pad 25: (no net) -> Net-(IC2-Pad25)
- IC2 pad 26: (no net) -> /USB2/USB2_REFCLK
- IC3 pad 6: (no net) -> /EEPROM/EEPROM_SCL
- IC3 pad 7: (no net) -> /EEPROM/EEPROM_WC
- IC4 pad 1: (no net) -> Net-(IC4-Pad1)
- IC4 pad 5: (no net) -> Net-(IC4-Pad5)
- IC4 pad 6: (no net) -> Net-(IC4-Pad6)
- IC7 pad 1: (no net) -> Net-(IC7-Pad1)
- IC7 pad 2: (no net) -> Net-(IC7-Pad2)
- IC7 pad 3: (no net) -> Net-(IC7-Pad3)
- IC7 pad 7: (no net) -> Net-(IC7-Pad7)
- IC9 pad A1: (no net) -> Net-(IC9-PadA1)
- IC9 pad A7: (no net) -> Net-(IC9-PadA7)
- IC9 pad B1: (no net) -> Net-(IC9-PadB1)
- IC9 pad B7: (no net) -> Net-(IC9-PadB7)
- IC9 pad C1: (no net) -> Net-(IC9-PadC1)
- IC9 pad C4: (no net) -> Net-(IC9-PadC4)
- IC9 pad C7: (no net) -> Net-(IC9-PadC7)
- IC9 pad D1: (no net) -> Net-(IC9-PadD1)
- IC9 pad D7: (no net) -> Net-(IC9-PadD7)
- IC9 pad E1: (no net) -> Net-(IC9-PadE1)
- IC9 pad E7: (no net) -> Net-(IC9-PadE7)
- IC9 pad F1: (no net) -> Net-(IC9-PadF1)
- IC9 pad F7: (no net) -> Net-(IC9-PadF7)
- IC9 pad G1: (no net) -> Net-(IC9-PadG1)
- IC9 pad G7: (no net) -> Net-(IC9-PadG7)
- IC9 pad H1: (no net) -> Net-(IC9-PadH1)
- IC9 pad H7: (no net) -> Net-(IC9-PadH7)
- IC9 pad J1: (no net) -> Net-(IC9-PadJ1)
- IC9 pad J7: (no net) -> Net-(IC9-PadJ7)
- IC9 pad K1: (no net) -> Net-(IC9-PadK1)
- IC9 pad K7: (no net) -> Net-(IC9-PadK7)
- IC9 pad L1: (no net) -> Net-(IC9-PadL1)
- IC9 pad L7: (no net) -> Net-(IC9-PadL7)
- IC9 pad M1: (no net) -> Net-(IC9-PadM1)
- IC9 pad M7: (no net) -> Net-(IC9-PadM7)
- IC9 pad N1: (no net) -> Net-(IC9-PadN1)
- IC9 pad N7: (no net) -> Net-(IC9-PadN7)
- IC9 pad P1: (no net) -> Net-(IC9-PadP1)
- IC9 pad P7: (no net) -> Net-(IC9-PadP7)
- IC9 pad R1: (no net) -> Net-(IC9-PadR1)
- IC9 pad R4: (no net) -> Net-(IC9-PadR4)
- IC9 pad R7: (no net) -> Net-(IC9-PadR7)
- IC9 pad T1: (no net) -> Net-(IC9-PadT1)
- IC9 pad T7: (no net) -> Net-(IC9-PadT7)
- IC9 pad U1: (no net) -> Net-(IC9-PadU1)
- IC9 pad U7: (no net) -> Net-(IC9-PadU7)
- J11 pad 5: (no net) -> /USB3/SSRX-
- J11 pad 6: (no net) -> /USB3/SSRX+
- J21 pad 2: (no net) -> Net-(J21-Pad2)
- J21 pad 5: (no net) -> Net-(J21-Pad5)
- J21 pad 6: (no net) -> Net-(J21-Pad6)
- J21 pad 9: (no net) -> Net-(J21-Pad9)
- J3 pad 1: (no net) -> /BTB_Connector/V1_MIX_SWITCH
- J3 pad 10: (no net) -> /BTB_Connector/OFFSET_DAC_LDAC
- J3 pad 11: (no net) -> /BTB_Connector/I2C1_SCL
- J3 pad 12: (no net) -> /BTB_Connector/OFFSET_DAC_RESET
- J3 pad 13: (no net) -> /BTB_Connector/I2C1_SDA
- J3 pad 14: (no net) -> /BTB_Connector/PORT_EXPANDER_DATA_INPUT
- J3 pad 15: (no net) -> GNDPWR
- J3 pad 16: (no net) -> /BTB_Connector/PORT_EXPANDER_DATA_OUTPUT
- J3 pad 17: (no net) -> Net-(J3-Pad17)
- J3 pad 18: (no net) -> /BTB_Connector/PORT_EXPANDER_SCK
- J3 pad 19: (no net) -> Net-(J3-Pad19)
- J3 pad 2: (no net) -> /BTB_Connector/OFFSET_DAC_MOSI
- J3 pad 20: (no net) -> /BTB_Connector/PORT_EXPANDER_CS
- J3 pad 21: (no net) -> Net-(J3-Pad21)
- J3 pad 22: (no net) -> Net-(J3-Pad22)
- J3 pad 23: (no net) -> Net-(J3-Pad23)
- J3 pad 24: (no net) -> Net-(J3-Pad24)
- J3 pad 25: (no net) -> Net-(J3-Pad25)
- J3 pad 26: (no net) -> Net-(J3-Pad26)
- J3 pad 27: (no net) -> Net-(J3-Pad27)
- J3 pad 28: (no net) -> Net-(J3-Pad28)
- J3 pad 29: (no net) -> Net-(J3-Pad29)
- J3 pad 30: (no net) -> Net-(J3-Pad30)
- J3 pad 31: (no net) -> Net-(J3-Pad31)
- J3 pad 32: (no net) -> Net-(J3-Pad32)
- J3 pad 33: (no net) -> Net-(J3-Pad33)
- J3 pad 34: (no net) -> Net-(J3-Pad34)
- J3 pad 35: (no net) -> Net-(J3-Pad35)
- J3 pad 36: (no net) -> Net-(J3-Pad36)
- J3 pad 37: (no net) -> Net-(J3-Pad37)
- J3 pad 38: (no net) -> Net-(J3-Pad38)
- J3 pad 39: (no net) -> Net-(J3-Pad39)
- J3 pad 4: (no net) -> /BTB_Connector/OFFSET_DAC_SCLK
- J3 pad 40: (no net) -> Net-(J3-Pad40)
- J3 pad 41: (no net) -> Net-(J3-Pad41)
- J3 pad 42: (no net) -> Net-(J3-Pad42)
- J3 pad 43: (no net) -> Net-(J3-Pad43)
- J3 pad 44: (no net) -> Net-(J3-Pad44)
- J3 pad 45: (no net) -> Net-(J3-Pad45)
- J3 pad 46: (no net) -> Net-(J3-Pad46)
- J3 pad 47: (no net) -> Net-(J3-Pad47)
- J3 pad 48: (no net) -> Net-(J3-Pad48)
- J3 pad 49: (no net) -> Net-(J3-Pad49)
- J3 pad 5: (no net) -> /BTB_Connector/V2_MIX_SWITCH
- J3 pad 50: (no net) -> Net-(J3-Pad50)
- J3 pad 51: (no net) -> Net-(J3-Pad51)
- J3 pad 52: (no net) -> Net-(J3-Pad52)
- J3 pad 53: (no net) -> Net-(J3-Pad53)
- J3 pad 54: (no net) -> Net-(J3-Pad54)
- J3 pad 55: (no net) -> Net-(J3-Pad55)
- J3 pad 56: (no net) -> Net-(J3-Pad56)
- J3 pad 57: (no net) -> Net-(J3-Pad57)
- J3 pad 58: (no net) -> Net-(J3-Pad58)
- J3 pad 59: (no net) -> Net-(J3-Pad59)
- J3 pad 6: (no net) -> /BTB_Connector/OFFSET_DAC_SS
- J3 pad 60: (no net) -> Net-(J3-Pad60)
- J3 pad 61: (no net) -> Net-(J3-Pad61)
- J3 pad 62: (no net) -> Net-(J3-Pad62)
- J3 pad 63: (no net) -> /FPGA_Banks/DAC_DCLK_OUT_N
- J3 pad 64: (no net) -> Net-(J3-Pad64)
- J3 pad 65: (no net) -> /FPGA_Banks/DAC_DCLK_OUT_P
- J3 pad 66: (no net) -> Net-(J3-Pad66)
- J3 pad 67: (no net) -> Net-(J3-Pad67)
- J3 pad 68: (no net) -> Net-(J3-Pad68)
- J3 pad 69: (no net) -> /FPGA_Banks/DAC_DCLK_IN_N
- J3 pad 70: (no net) -> Net-(J3-Pad70)
- J3 pad 71: (no net) -> /FPGA_Banks/DAC_DCLK_IN_P
- J3 pad 72: (no net) -> Net-(J3-Pad72)
- J3 pad 73: (no net) -> Net-(J3-Pad73)
- J3 pad 74: (no net) -> Net-(J3-Pad74)
- J3 pad 75: (no net) -> /FDAC_CLKIN_N
- J3 pad 76: (no net) -> Net-(J3-Pad76)
- J3 pad 77: (no net) -> /FDAC_CLKIN_P
- J3 pad 78: (no net) -> Net-(J3-Pad78)
- J3 pad 79: (no net) -> Net-(J3-Pad79)
- J3 pad 8: (no net) -> /BTB_Connector/OFFSET_DAC_MISO
- J3 pad 80: (no net) -> Net-(J3-Pad80)
- J3 pad 9: (no net) -> /BTB_Connector/FALSE_SUM_OUTPUT_BTB
- J4 pad 10: (no net) -> /BTB_Connector/FDAC_DB14_P
- J4 pad 11: (no net) -> /BTB_Connector/FDAC_DB6_P
- J4 pad 12: (no net) -> /BTB_Connector/FDAC_DB14_N
- J4 pad 15: (no net) -> /BTB_Connector/FDAC_DB5_N
- J4 pad 16: (no net) -> /BTB_Connector/FDAC_DB13_P
- J4 pad 17: (no net) -> /BTB_Connector/FDAC_DB5_P
- J4 pad 18: (no net) -> /BTB_Connector/FDAC_DB13_N
- J4 pad 21: (no net) -> /BTB_Connector/FDAC_DB4_N
- J4 pad 22: (no net) -> /BTB_Connector/FDAC_DB12_P
- J4 pad 23: (no net) -> /BTB_Connector/FDAC_DB4_P
- J4 pad 24: (no net) -> /BTB_Connector/FDAC_DB12_N
- J4 pad 27: (no net) -> /BTB_Connector/FDAC_DB3_N
- J4 pad 28: (no net) -> /BTB_Connector/FDAC_DB11_P
- J4 pad 29: (no net) -> /BTB_Connector/FDAC_DB3_P
- J4 pad 3: (no net) -> /BTB_Connector/FDAC_DB7_N
- J4 pad 30: (no net) -> /BTB_Connector/FDAC_DB11_N
- J4 pad 33: (no net) -> /BTB_Connector/FDAC_DB2_N
- J4 pad 34: (no net) -> /BTB_Connector/FDAC_DB10_P
- J4 pad 35: (no net) -> /BTB_Connector/FDAC_DB2_P
- J4 pad 36: (no net) -> /BTB_Connector/FDAC_DB10_N
- J4 pad 39: (no net) -> /BTB_Connector/FDAC_DB1_N
- J4 pad 4: (no net) -> /BTB_Connector/FDAC_DB15_P
- J4 pad 40: (no net) -> /BTB_Connector/FDAC_DB9_P
- J4 pad 41: (no net) -> /BTB_Connector/FDAC_DB1_P
- J4 pad 42: (no net) -> /BTB_Connector/FDAC_DB9_N
- J4 pad 45: (no net) -> /BTB_Connector/FDAC_DB0_N
- J4 pad 46: (no net) -> /BTB_Connector/FDAC_DB8_P
- J4 pad 47: (no net) -> /BTB_Connector/FDAC_DB0_P
- J4 pad 48: (no net) -> /BTB_Connector/FDAC_DB8_N
- J4 pad 5: (no net) -> /BTB_Connector/FDAC_DB7_P
- J4 pad 51: (no net) -> /BTB_Connector/ADC1_CLK_P
- J4 pad 52: (no net) -> /BTB_Connector/ADC_CNV_N
- J4 pad 53: (no net) -> /BTB_Connector/ADC1_CLK_N
- J4 pad 54: (no net) -> /BTB_Connector/ADC_CNV_P
- J4 pad 57: (no net) -> /BTB_Connector/ADC1_DCO_P
- J4 pad 58: (no net) -> /BTB_Connector/ADC3_DA_N
- J4 pad 59: (no net) -> /BTB_Connector/ADC1_DCO_N
- J4 pad 6: (no net) -> /BTB_Connector/FDAC_DB15_N
- J4 pad 60: (no net) -> /BTB_Connector/ADC3_DA_P
- J4 pad 63: (no net) -> /BTB_Connector/ADC1_DA_P
- J4 pad 64: (no net) -> /BTB_Connector/ADC3_DCO_N
- J4 pad 65: (no net) -> /BTB_Connector/ADC1_DA_N
- J4 pad 66: (no net) -> /BTB_Connector/ADC3_DCO_P
- J4 pad 69: (no net) -> /BTB_Connector/ADC2_CLK_P
- J4 pad 70: (no net) -> /BTB_Connector/ADC3_CLK_N
- J4 pad 71: (no net) -> /BTB_Connector/ADC2_CLK_N
- J4 pad 72: (no net) -> /BTB_Connector/ADC3_CLK_P
- J4 pad 75: (no net) -> /BTB_Connector/ADC2_DCO_P
- J4 pad 76: (no net) -> /BTB_Connector/ADC2_DA_N
- J4 pad 77: (no net) -> /BTB_Connector/ADC2_DCO_N
- J4 pad 78: (no net) -> /BTB_Connector/ADC2_DA_P
- J4 pad 9: (no net) -> /BTB_Connector/FDAC_DB6_N
- J7 pad 1: /RTC_FAN/12VIN -> /12V
- R100 pad 1: (no net) -> Net-(R100-Pad1)
- R105 pad 1: (no net) -> Net-(R105-Pad1)
- R106 pad 1: (no net) -> Net-(R106-Pad1)
- R117 pad 2: (no net) -> Net-(J12-Pad1)
- R119 pad 1: (no net) -> Net-(J13-Pad1)
- R12 pad 2: (no net) -> Net-(D3-Pad2)
- R120 pad 1: (no net) -> Net-(R120-Pad1)
- R121 pad 1: (no net) -> Net-(R121-Pad1)
- R124 pad 2: (no net) -> Net-(J14-Pad1)
- R126 pad 2: (no net) -> Net-(R126-Pad2)
- R129 pad 2: (no net) -> /FPGA_Banks/LED1
- R131 pad 1: (no net) -> Net-(D11-Pad1)
- R15 pad 2: /Clock_Gen/CG_SDA -> /I2C2_SDA
- R18 pad 2: /Clock_Gen/CG_SCL -> /I2C_SCL
- R181 pad 1: (no net) -> Net-(J20-Pad14)
- R182 pad 1: (no net) -> Net-(J20-Pad16)
- R185 pad 2: (no net) -> Net-(R185-Pad2)
- R32 pad 2: (no net) -> Net-(C111-Pad1)
- R37 pad 2: /RTC_FAN/RTC_SDA -> /I2C2_SDA
- R40 pad 1: (no net) -> /FPGA_Banks/FAN_CTRL_PWM
- R86 pad 1: (no net) -> Net-(R86-Pad1)
- R87 pad 1: (no net) -> Net-(R87-Pad1)
- R88 pad 1: (no net) -> Net-(R88-Pad1)
- R88 pad 2: (no net) -> /USB3/CTL4
- R89 pad 1: (no net) -> Net-(R89-Pad1)
- R90 pad 1: (no net) -> Net-(R90-Pad1)
- R91 pad 1: (no net) -> Net-(R91-Pad1)
- R92 pad 1: (no net) -> Net-(R92-Pad1)
- R93 pad 1: (no net) -> Net-(R93-Pad1)
- R93 pad 2: (no net) -> /USB3/CTL3
- R94 pad 1: (no net) -> Net-(R94-Pad1)
- R95 pad 1: (no net) -> Net-(R95-Pad1)
- R96 pad 1: (no net) -> Net-(R96-Pad1)
- R97 pad 1: (no net) -> Net-(R97-Pad1)
- R98 pad 1: (no net) -> Net-(R98-Pad1)
- U1 pad A20: (no net) -> /BTB_Connector/FDAC_DB14_N
- U1 pad A5: (no net) -> Net-(U1-PadA5)
- U1 pad A6: (no net) -> Net-(U1-PadA6)
- U1 pad A7: (no net) -> Net-(U1-PadA7)
- U1 pad A9: (no net) -> Net-(U1-PadA9)
- U1 pad B10: (no net) -> Net-(U1-PadB10)
- U1 pad B12: (no net) -> Net-(U1-PadB12)
- U1 pad B13: (no net) -> Net-(U1-PadB13)
- U1 pad B14: (no net) -> Net-(U1-PadB14)
- U1 pad B15: (no net) -> Net-(U1-PadB15)
- U1 pad B19: (no net) -> /BTB_Connector/FDAC_DB14_P
- U1 pad B20: (no net) -> /BTB_Connector/FDAC_DB15_N
- U1 pad B5: (no net) -> Net-(U1-PadB5)
- U1 pad B7: (no net) -> Net-(U1-PadB7)
- U1 pad B8: (no net) -> Net-(U1-PadB8)
- U1 pad B9: (no net) -> Net-(U1-PadB9)
- U1 pad C12: (no net) -> Net-(U1-PadC12)
- U1 pad C17: (no net) -> Net-(U1-PadC17)
- U1 pad C20: (no net) -> /BTB_Connector/FDAC_DB15_P
- U1 pad C5: (no net) -> Net-(U1-PadC5)
- U1 pad C6: (no net) -> Net-(U1-PadC6)
- U1 pad C7: (no net) -> Net-(U1-PadC7)
- U1 pad C8: (no net) -> Net-(U1-PadC8)
- U1 pad D18: (no net) -> /BTB_Connector/FDAC_DB13_N
- U1 pad D19: (no net) -> /FPGA_Banks/FX3_DQ11
- U1 pad D20: (no net) -> /FPGA_Banks/FX3_DQ12
- U1 pad D5: (no net) -> Net-(U1-PadD5)
- U1 pad D6: (no net) -> Net-(U1-PadD6)
- U1 pad D8: (no net) -> Net-(U1-PadD8)
- U1 pad D9: (no net) -> Net-(U1-PadD9)
- U1 pad E11: (no net) -> Net-(U1-PadE11)
- U1 pad E12: (no net) -> Net-(U1-PadE12)
- U1 pad E17: (no net) -> /BTB_Connector/FDAC_DB13_P
- U1 pad E18: (no net) -> /FPGA_Banks/FX3_DQ23
- U1 pad E19: (no net) -> /FPGA_Banks/FX3_DQ24
- U1 pad E6: (no net) -> Net-(U1-PadE6)
- U1 pad E7: (no net) -> Net-(U1-PadE7)
- U1 pad E8: (no net) -> Net-(U1-PadE8)
- U1 pad E9: (no net) -> Net-(U1-PadE9)
- U1 pad F13: (no net) -> Net-(U1-PadF13)
- U1 pad F16: (no net) -> /BTB_Connector/FDAC_DB12_P
- U1 pad F17: (no net) -> /BTB_Connector/FDAC_DB12_N
- U1 pad F19: (no net) -> /FPGA_Banks/FX3_DQ21
- U1 pad F20: (no net) -> /FPGA_Banks/FX3_DQ22
- U1 pad G14: (no net) -> Net-(U1-PadG14)
- U1 pad G15: (no net) -> /BTB_Connector/FDAC_DB2_P
- U1 pad G17: (no net) -> /FPGA_Banks/FX3_CTL5
- U1 pad G18: (no net) -> /FPGA_Banks/FX3_CTL6
- U1 pad G19: (no net) -> /FPGA_Banks/FX3_CTL11
- U1 pad G20: (no net) -> /FPGA_Banks/FX3_CTL12
- U1 pad H15: (no net) -> /BTB_Connector/FDAC_DB2_N
- U1 pad H16: (no net) -> /FPGA_Banks/DAC_DCLK_IN_P
- U1 pad H17: (no net) -> /FPGA_Banks/DAC_DCLK_IN_N
- U1 pad H18: (no net) -> /FPGA_Banks/FX3_I2S_MCLK
- U1 pad H20: (no net) -> /FPGA_Banks/FX3_I2S_WS
- U1 pad J14: (no net) -> /FPGA_Banks/FX3_CTL4
- U1 pad J15: (no net) -> Net-(U1-PadJ15)
- U1 pad J16: (no net) -> /BTB_Connector/FDAC_DB10_N
- U1 pad J18: (no net) -> /FPGA_Banks/FX3_I2S_SD
- U1 pad J19: (no net) -> /FPGA_Banks/FX3_DQ16
- U1 pad J20: (no net) -> /FPGA_Banks/FX3_I2S_CLK
- U1 pad K14: (no net) -> /FPGA_Banks/FX3_CTL3
- U1 pad K16: (no net) -> /BTB_Connector/FDAC_DB10_P
- U1 pad K17: (no net) -> /FPGA_Banks/DAC_DCLK_OUT_P
- U1 pad K18: (no net) -> /FPGA_Banks/DAC_DCLK_OUT_N
- U1 pad K19: (no net) -> /FPGA_Banks/FX3_DQ15
- U1 pad L14: (no net) -> /FPGA_Banks/FX3_CTL1
- U1 pad L15: (no net) -> /FPGA_Banks/FX3_CTL2
- U1 pad L16: (no net) -> /FPGA_Banks/FX3_CTL7
- U1 pad L17: (no net) -> /FPGA_Banks/FX3_CTL8
- U1 pad L19: (no net) -> /FPGA_Banks/FX3_DQ17
- U1 pad L20: (no net) -> /FPGA_Banks/FX3_DQ18
- U1 pad M14: (no net) -> /BTB_Connector/FDAC_DB11_P
- U1 pad M15: (no net) -> /BTB_Connector/FDAC_DB11_N
- U1 pad M17: (no net) -> /FPGA_Banks/FX3_CTL9
- U1 pad M18: (no net) -> /FPGA_Banks/FX3_CTL10
- U1 pad M19: (no net) -> /FPGA_Banks/FX3_DQ19
- U1 pad M20: (no net) -> /FPGA_Banks/FX3_DQ20
- U1 pad N15: (no net) -> /FPGA_Banks/FX3_DQ13
- U1 pad N16: (no net) -> /FPGA_Banks/FX3_DQ14
- U1 pad N17: (no net) -> /BTB_Connector/FDAC_DB6_P
- U1 pad N18: (no net) -> /FPGA_Banks/FX3_PCLK
- U1 pad N20: (no net) -> /BTB_Connector/FDAC_DB0_P
- U1 pad P14: (no net) -> /BTB_Connector/FDAC_DB4_P
- U1 pad P15: (no net) -> /BTB_Connector/FDAC_DB5_P
- U1 pad P16: (no net) -> /BTB_Connector/FDAC_DB5_N
- U1 pad P18: (no net) -> /BTB_Connector/FDAC_DB6_N
- U1 pad P19: (no net) -> /FPGA_Banks/FX3_DQ0
- U1 pad P20: (no net) -> /BTB_Connector/FDAC_DB0_N
- U1 pad R14: (no net) -> /BTB_Connector/FDAC_DB4_N
- U1 pad R16: (no net) -> /BTB_Connector/FDAC_DB3_P
- U1 pad R17: (no net) -> /BTB_Connector/FDAC_DB3_N
- U1 pad R18: (no net) -> /FPGA_Banks/FX3_DQ2
- U1 pad R19: (no net) -> Net-(U1-PadR19)
- U1 pad T10: (no net) -> /BTB_Connector/FDAC_DB9_N
- U1 pad T11: (no net) -> /BTB_Connector/FDAC_DB9_P
- U1 pad T12: (no net) -> /FPGA_Banks/FX3_DQ9
- U1 pad T14: (no net) -> /FPGA_Banks/FX3_DQ7
- U1 pad T15: (no net) -> /FPGA_Banks/FX3_DQ8
- U1 pad T16: (no net) -> /FPGA_Banks/FX3_DQ31
- U1 pad T17: (no net) -> /FPGA_Banks/FX3_DQ1
- U1 pad T19: (no net) -> Net-(U1-PadT19)
- U1 pad T20: (no net) -> /FPGA_Banks/FX3_DQ3
- U1 pad T5: (no net) -> /BTB_Connector/ADC2_CLK_P
- U1 pad T9: (no net) -> Net-(U1-PadT9)
- U1 pad U10: (no net) -> Net-(U1-PadU10)
- U1 pad U12: (no net) -> /FPGA_Banks/FX3_DQ10
- U1 pad U14: (no net) -> /BTB_Connector/FDAC_DB1_P
- U1 pad U15: (no net) -> /BTB_Connector/FDAC_DB1_N
- U1 pad U17: (no net) -> /FPGA_Banks/FX3_CTL0
- U1 pad U18: (no net) -> Net-(U1-PadU18)
- U1 pad U19: (no net) -> Net-(U1-PadU19)
- U1 pad U20: (no net) -> /FPGA_Banks/FX3_DQ4
- U1 pad U5: (no net) -> /BTB_Connector/ADC2_CLK_N
- U1 pad U7: (no net) -> /BTB_Connector/ADC3_CLK_P
- U1 pad U8: (no net) -> /BTB_Connector/ADC1_DCO_N
- U1 pad U9: (no net) -> /BTB_Connector/ADC1_DCO_P
- U1 pad V10: (no net) -> /BTB_Connector/ADC2_DA_N
- U1 pad V11: (no net) -> /BTB_Connector/ADC2_DA_P
- U1 pad V12: (no net) -> /BTB_Connector/FDAC_DB8_P
- U1 pad V13: (no net) -> Net-(U1-PadV13)
- U1 pad V15: (no net) -> /FPGA_Banks/FX3_I2C_SDA
- U1 pad V16: (no net) -> /FPGA_Banks/FX3_DQ29
- U1 pad V17: (no net) -> /FPGA_Banks/FX3_DQ5
- U1 pad V18: (no net) -> /FPGA_Banks/FX3_DQ6
- U1 pad V20: (no net) -> /FPGA_Banks/FX3_DQ25
- U1 pad V5: (no net) -> Net-(U1-PadV5)
- U1 pad V6: (no net) -> /BTB_Connector/ADC3_DA_P
- U1 pad V7: (no net) -> /BTB_Connector/ADC3_CLK_N
- U1 pad V8: (no net) -> /BTB_Connector/ADC_CNV_P
- U1 pad W10: (no net) -> /BTB_Connector/ADC1_CLK_P
- U1 pad W11: (no net) -> /BTB_Connector/ADC1_DA_P
- U1 pad W13: (no net) -> /BTB_Connector/FDAC_DB8_N
- U1 pad W14: (no net) -> /FPGA_Banks/FX3_DQ27
- U1 pad W15: (no net) -> /FPGA_Banks/FX3_I2C_SCL
- U1 pad W16: (no net) -> /FPGA_Banks/FX3_DQ30
- U1 pad W18: (no net) -> /BTB_Connector/FDAC_DB7_P
- U1 pad W19: (no net) -> /BTB_Connector/FDAC_DB7_N
- U1 pad W20: (no net) -> /FPGA_Banks/FX3_DQ26
- U1 pad W6: (no net) -> /BTB_Connector/ADC3_DA_N
- U1 pad W8: (no net) -> /BTB_Connector/ADC_CNV_N
- U1 pad W9: (no net) -> /BTB_Connector/ADC1_CLK_N
- U1 pad Y11: (no net) -> /BTB_Connector/ADC1_DA_N
- U1 pad Y12: (no net) -> /BTB_Connector/ADC2_DCO_P
- U1 pad Y13: (no net) -> /BTB_Connector/ADC2_DCO_N
- U1 pad Y14: (no net) -> /FPGA_Banks/FX3_DQ28
- U1 pad Y18: (no net) -> /FPGA_Banks/FX3_PMOD2
- U1 pad Y19: (no net) -> /FPGA_Banks/FX3_INT_N_CTL15
- U1 pad Y6: (no net) -> Net-(U1-PadY6)
- U1 pad Y7: (no net) -> Net-(U1-PadY7)
- U1 pad Y8: (no net) -> /BTB_Connector/ADC3_DCO_N
- U1 pad Y9: (no net) -> /BTB_Connector/ADC3_DCO_P
- U13 pad 1: (no net) -> /LED_Comm/SCL
- U13 pad 4: (no net) -> /I2C_SCL
- U13 pad 5: (no net) -> /I2C2_SDA
- U13 pad 8: (no net) -> /LED_Comm/SDA
- U14 pad 1: (no net) -> /FPGA_Banks/F_UART_TX
- U14 pad 12: (no net) -> /LED_Comm/SPI_SS
- U14 pad 13: (no net) -> /LED_Comm/SPI_CLK
- U14 pad 14: (no net) -> /LED_Comm/SPI_MOSI
- U14 pad 15: (no net) -> /LED_Comm/SPI_MISO
- U14 pad 16: (no net) -> Net-(U14-Pad16)
- U14 pad 17: (no net) -> Net-(U14-Pad17)
- U14 pad 18: (no net) -> /LED_Comm/UART_RX
- U14 pad 20: (no net) -> /LED_Comm/UART_TX
- U14 pad 3: (no net) -> /FPGA_Banks/F_UART_RX
- U14 pad 4: (no net) -> Net-(U14-Pad4)
- U14 pad 5: (no net) -> Net-(U14-Pad5)
- U14 pad 6: (no net) -> /FPGA_Banks/F_SPI_MISO
- U14 pad 7: (no net) -> /FPGA_Banks/F_SPI_MOSI
- U14 pad 8: (no net) -> /FPGA_Banks/F_SPI_CLK
- U14 pad 9: (no net) -> /FPGA_Banks/F_SPI_SS
- U15 pad 1: (no net) -> /FPGA_Banks/F_CAN_H
- U15 pad 12: (no net) -> Net-(U15-Pad12)
- U15 pad 13: (no net) -> Net-(U15-Pad13)
- U15 pad 14: (no net) -> Net-(U15-Pad14)
- U15 pad 15: (no net) -> /LED_Comm/LCD_RX
- U15 pad 16: (no net) -> /LED_Comm/LCD_TX
- U15 pad 17: (no net) -> /LED_Comm/LCD_RESET
- U15 pad 18: (no net) -> /LED_Comm/CAN_L
- U15 pad 20: (no net) -> /LED_Comm/CAN_H
- U15 pad 3: (no net) -> /FPGA_Banks/F_CAN_L
- U15 pad 4: (no net) -> /FPGA_Banks/F_LCD_RESET
- U15 pad 5: (no net) -> /FPGA_Banks/F_LCD_TX
- U15 pad 6: (no net) -> /FPGA_Banks/F_LCD_RX
- U15 pad 7: (no net) -> Net-(U15-Pad7)
- U15 pad 8: (no net) -> Net-(U15-Pad8)
- U15 pad 9: (no net) -> Net-(U15-Pad9)
- U16 pad J1: (no net) -> Net-(U16-PadJ1)
- U16 pad J9: (no net) -> Net-(U16-PadJ9)
- U16 pad L1: (no net) -> Net-(U16-PadL1)
- U16 pad L9: (no net) -> Net-(U16-PadL9)
- U16 pad M7: (no net) -> Net-(U16-PadM7)
- U17 pad J1: (no net) -> Net-(U17-PadJ1)
- U17 pad J9: (no net) -> Net-(U17-PadJ9)
- U17 pad L1: (no net) -> Net-(U17-PadL1)
- U17 pad L9: (no net) -> Net-(U17-PadL9)
- U17 pad M7: (no net) -> Net-(U17-PadM7)
- U18 pad 1: (no net) -> /Ethernet/ETH_PHY_CONN/ETH_A_P
- U18 pad 10: (no net) -> /Ethernet/ETH_PHY_CONN/ETH_D_P
- U18 pad 11: (no net) -> /Ethernet/ETH_PHY_CONN/ETH_D_N
- U18 pad 13: (no net) -> Net-(U18-Pad13)
- U18 pad 14: (no net) -> Net-(U18-Pad14)
- U18 pad 15: (no net) -> Net-(U18-Pad15)
- U18 pad 16: (no net) -> Net-(U18-Pad16)
- U18 pad 17: (no net) -> Net-(U18-Pad17)
- U18 pad 2: (no net) -> /Ethernet/ETH_PHY_CONN/ETH_A_N
- U18 pad 4: (no net) -> /Ethernet/ETH_PHY_CONN/ETH_B_P
- U18 pad 40: (no net) -> Net-(U18-Pad40)
- U18 pad 48: (no net) -> Net-(U18-Pad48)
- U18 pad 5: (no net) -> /Ethernet/ETH_PHY_CONN/ETH_B_N
- U18 pad 7: (no net) -> /Ethernet/ETH_PHY_CONN/ETH_C_P
- U18 pad 8: (no net) -> /Ethernet/ETH_PHY_CONN/ETH_C_N
- U2 pad 12: (no net) -> /Clock_Gen/CG_OEB
- U2 pad 13: /Clock_Gen/CG_SDA -> /I2C2_SDA
- U2 pad 14: /Clock_Gen/CG_SCL -> /I2C_SCL
- U2 pad 17: (no net) -> /Clock_Gen/CG_RSTB
- U2 pad 22: (no net) -> Net-(U2-Pad22)
- U2 pad 27: (no net) -> /Clock_Gen/CG_LOLB
- U2 pad 28: (no net) -> Net-(U2-Pad28)
- U2 pad 3: (no net) -> /Clock_Gen/CG_IN_SEL0
- U2 pad 33: (no net) -> /Clock_Gen/CG_INTRB
- U2 pad 37: (no net) -> /Clock_Gen/CG_IN_SEL1
- U4 pad 15: /RTC_FAN/RTC_SDA -> /I2C2_SDA
- U4 pad 4: (no net) -> /RTC_FAN/RTC_RST
- U6 pad 12: (no net) -> Net-(U6-Pad12)
- U6 pad 3: (no net) -> Net-(C137-Pad2)
- U8 pad 4: (no net) -> /USB3/USB3_D+
- U8 pad 6: (no net) -> /USB3/USB3_D-
- Y2 pad 2: (no net) -> Net-(Y2-Pad2)
- Y2 pad 4: (no net) -> Net-(Y2-Pad4)
